File: rev1/pcb/tako.kicad_pcb (KiCad board)
At the start: 2 copper layers, 252.1 x 110.4 mm, 124 parts, among them J1 MJ-4PP-9, J101 MJ-4PP-9, SW1 EC_SW, SW10 EC_SW, SW101 EC_SW, SW102 EC_SW, SW103 EC_SW, SW104 EC_SW, SW105 EC_SW, SW106 EC_SW, SW107 EC_SW, SW108 EC_SW, SW109 EC_SW, SW11 EC_SW, SW110 EC_SW, SW111 EC_SW, SW112 EC_SW, SW113 EC_SW, SW114 EC_SW, SW115 EC_SW, SW116 EC_SW, SW117 EC_SW, SW118 EC_SW, SW12 EC_SW, SW13 EC_SW, SW14 EC_SW, SW15 EC_SW, SW16 EC_SW, SW17 EC_SW, SW18 EC_SW, SW2 EC_SW, SW3 EC_SW, SW4 EC_SW, SW5 EC_SW, SW6 EC_SW, SW7 EC_SW, SW8 EC_SW, SW9 EC_SW, U1 STeMCell, U101 STeMCell, U102 74HC4051, U103 OPA350, U2 74HC4051, U3 OPA350

Commit message: updated holes for 4.5mm standoff
Parts:
- H1, H10, H101, H102, H103, H104, H105, H106, H107, H108, H109, H11, H110, H111, H112, H113, H114, H12, H13, H14, H18, H19, H2, H3, H4, H5, H6, H7, H8, H9: footprint tako:MountingHole_3.4mm -> MountingHole:MountingHole_4.5mm
Routing:
- net COL1_R: track 186.9 -> 186.2 mm
- net +3.3V: track 52.6 -> 52.0 mm
