File: rev1/pcb/tako_left.kicad_pcb (KiCad board)
At the start: 2 copper layers, 124.7 x 110.4 mm, 61 parts, among them J101 MJ-4PP-9, SW101 EC_SW, SW102 EC_SW, SW103 EC_SW, SW104 EC_SW, SW105 EC_SW, SW106 EC_SW, SW107 EC_SW, SW108 EC_SW, SW109 EC_SW, SW110 EC_SW, SW111 EC_SW, SW112 EC_SW, SW113 EC_SW, SW114 EC_SW, SW115 EC_SW, SW116 EC_SW, SW117 EC_SW, SW118 EC_SW, U101 STeMCell, U102 74HC4051, U103 OPA350

Commit message: updated holes for 4.5mm standoff
Parts:
- removed BAT_HOLE+101: MountingHole_Pad, tako:bat_pin+
- removed BAT_HOLE-101: MountingHole_Pad, tako:bat_pin-
- removed C101, C103: 100n, Capacitor_SMD:C_0805_2012Metric_Pad1.18x1.45mm_HandSolder
- removed C102: 220p, Capacitor_SMD:C_0805_2012Metric_Pad1.18x1.45mm_HandSolder
- removed DISP101: nice!view, tako:nice_view
- removed H101, H102, H103, H104, H105, H106, H107, H108, H109, H110, H111, H112, H113, H114, H18: MountingHole, tako:MountingHole_3.4mm
- removed H115, H116, H117: MountingHole, tako:M2_hole_3.5mm
- removed J101: MJ-4PP-9, tako:TRRS-PJ-320A
- removed JP101: Ext_Res, Resistor_SMD:R_0805_2012Metric_Pad1.20x1.40mm_HandSolder
- removed PSW101: SW_SPDT, tako:SW_SPDT_SMD_PCM12
- removed R101, R102, R103, R104: 100, Resistor_SMD:R_0805_2012Metric_Pad1.20x1.40mm_HandSolder
- removed R105, R106, R107, R108, R109, R110: 100k, Resistor_SMD:R_0805_2012Metric_Pad1.20x1.40mm_HandSolder
- removed R111: 1k, Resistor_SMD:R_0805_2012Metric_Pad1.20x1.40mm_HandSolder
- removed R112: 5.1k, Resistor_SMD:R_0805_2012Metric_Pad1.20x1.40mm_HandSolder
- removed RSW101: Reset, Button_Switch_SMD:Panasonic_EVQPUL_EVQPUC
- removed SW101, SW102, SW103, SW104, SW105, SW106, SW107, SW108, SW109, SW110, SW111, SW112, SW113, SW114, SW115: EC_SW, tako:ecs_pad_1U_no_ring
- removed SW116, SW117, SW118: EC_SW, tako:ecs_pad_1U_no_ring_90deg
- removed U101: STeMCell, tako:ArduinoProMicro
- removed U102: 74HC4051, Package_SO:SOIC-16_3.9x9.9mm_P1.27mm
- removed U103: OPA350, Package_SO:SOIC-8_3.9x4.9mm_P1.27mm
- added BAT_HOLE+1: MountingHole_Pad, tako:bat_pin+, F.Cu at (250.1, 57.8)
- added BAT_HOLE-1: MountingHole_Pad, tako:bat_pin-, F.Cu at (265.4, 57.8)
- added C1: 100n, Capacitor_SMD:C_0805_2012Metric_Pad1.18x1.45mm_HandSolder, F.Cu at (199.9, 95.9)
- added C2: 220p, Capacitor_SMD:C_0805_2012Metric_Pad1.18x1.45mm_HandSolder, F.Cu at (201.1, 101.5)
- added C3: 100n, Capacitor_SMD:C_0805_2012Metric_Pad1.18x1.45mm_HandSolder, F.Cu at (214.0, 97.6)
- added DISP1: nice!view, tako:nice_view, F.Cu at (257.8, 75.9)
- added H1: MountingHole, MountingHole:MountingHole_4.5mm, F.Cu at (162.6, 44.7)
- added H10: MountingHole, MountingHole:MountingHole_4.5mm, F.Cu at (238.8, 35.7)
- added H11: MountingHole, MountingHole:MountingHole_4.5mm, F.Cu at (238.8, 55.4)
- added H12: MountingHole, MountingHole:MountingHole_4.5mm, F.Cu at (238.8, 74.4)
- added H13: MountingHole, MountingHole:MountingHole_4.5mm, F.Cu at (239.3, 106.2)
- added H14: MountingHole, MountingHole:MountingHole_4.5mm, F.Cu at (274.7, 117.0)
- added H15: MountingHole, tako:M2_hole_3.5mm, F.Cu at (250.4, 54.5)
- added H16: MountingHole, tako:M2_hole_3.5mm, F.Cu at (265.1, 54.5)
- added H17: MountingHole, tako:M2_hole_3.5mm, F.Cu at (250.4, 97.0)
- added H19: MountingHole, MountingHole:MountingHole_4.5mm, F.Cu at (257.7, 116.7)
- added H2: MountingHole, MountingHole:MountingHole_4.5mm, F.Cu at (162.6, 64.4)
- added H3: MountingHole, MountingHole:MountingHole_4.5mm, F.Cu at (162.6, 83.4)
- added H4: MountingHole, MountingHole:MountingHole_4.5mm, F.Cu at (181.7, 32.7)
- added H5: MountingHole, MountingHole:MountingHole_4.5mm, F.Cu at (176.6, 95.0)
- added H6: MountingHole, MountingHole:MountingHole_4.5mm, F.Cu at (200.7, 46.4)
- added H7: MountingHole, MountingHole:MountingHole_4.5mm, F.Cu at (200.7, 65.4)
- added H8: MountingHole, MountingHole:MountingHole_4.5mm, F.Cu at (200.7, 87.0)
- added H9: MountingHole, MountingHole:MountingHole_4.5mm, F.Cu at (219.8, 33.2)
- added J1: MJ-4PP-9, tako:TRRS-PJ-320A, F.Cu at (266.7, 97.0)
- added JP1: Ext_Res, Resistor_SMD:R_0805_2012Metric_Pad1.20x1.40mm_HandSolder, F.Cu at (207.6, 95.9)
- added PSW1: SW_SPDT, tako:SW_SPDT_SMD_PCM12, B.Cu at (257.8, 58.1)
- added R1: 100, Resistor_SMD:R_0805_2012Metric_Pad1.20x1.40mm_HandSolder, B.Cu at (257.8, 62.2)
- added R10: 100k, Resistor_SMD:R_0805_2012Metric_Pad1.20x1.40mm_HandSolder, F.Cu at (207.6, 97.9)
- added R11: 1k, Resistor_SMD:R_0805_2012Metric_Pad1.20x1.40mm_HandSolder, F.Cu at (203.2, 96.9)
- added R12: 5.1k, Resistor_SMD:R_0805_2012Metric_Pad1.20x1.40mm_HandSolder, F.Cu at (243.4, 98.0)
- added R2: 100, Resistor_SMD:R_0805_2012Metric_Pad1.20x1.40mm_HandSolder, B.Cu at (257.8, 64.2)
- added R3: 100, Resistor_SMD:R_0805_2012Metric_Pad1.20x1.40mm_HandSolder, B.Cu at (257.8, 66.1)
- added R4: 100, Resistor_SMD:R_0805_2012Metric_Pad1.20x1.40mm_HandSolder, F.Cu at (241.5, 98.0)
- added R5: 100k, Resistor_SMD:R_0805_2012Metric_Pad1.20x1.40mm_HandSolder, F.Cu at (187.5, 95.6)
- added R6: 100k, Resistor_SMD:R_0805_2012Metric_Pad1.20x1.40mm_HandSolder, F.Cu at (183.2, 95.5)
- added R7: 100k, Resistor_SMD:R_0805_2012Metric_Pad1.20x1.40mm_HandSolder, F.Cu at (191.8, 95.6)
- added R8: 100k, Resistor_SMD:R_0805_2012Metric_Pad1.20x1.40mm_HandSolder, F.Cu at (178.3, 103.5)
- added R9: 100k, Resistor_SMD:R_0805_2012Metric_Pad1.20x1.40mm_HandSolder, F.Cu at (182.2, 99.6)
- added RSW1: Reset, Button_Switch_SMD:Panasonic_EVQPUL_EVQPUC, F.Cu at (265.1, 105.4)
- added SW1: EC_SW, tako:ecs_pad_1U_no_ring, F.Cu at (162.6, 54.9)
- added SW10: EC_SW, tako:ecs_pad_1U_no_ring, F.Cu at (238.8, 64.9)
- added SW11: EC_SW, tako:ecs_pad_1U_no_ring, F.Cu at (162.6, 93.0)
- added SW12: EC_SW, tako:ecs_pad_1U_no_ring, F.Cu at (181.7, 81.0)
- added SW13: EC_SW, tako:ecs_pad_1U_no_ring, F.Cu at (200.7, 75.0)
- added SW14: EC_SW, tako:ecs_pad_1U_no_ring, F.Cu at (219.8, 81.5)
- added SW15: EC_SW, tako:ecs_pad_1U_no_ring, F.Cu at (238.8, 84.0)
- added SW16: EC_SW, tako:ecs_pad_1U_no_ring_90deg, F.Cu at (265.2, 124.0)
- added SW17: EC_SW, tako:ecs_pad_1U_no_ring_90deg, F.Cu at (248.7, 111.5)
- added SW18: EC_SW, tako:ecs_pad_1U_no_ring_90deg, F.Cu at (228.9, 103.3)
- added SW2: EC_SW, tako:ecs_pad_1U_no_ring, F.Cu at (181.7, 42.9)
- added SW3: EC_SW, tako:ecs_pad_1U_no_ring, F.Cu at (200.7, 36.9)
- added SW4: EC_SW, tako:ecs_pad_1U_no_ring, F.Cu at (219.8, 43.4)
- added SW5: EC_SW, tako:ecs_pad_1U_no_ring, F.Cu at (238.8, 45.9)
- added SW6: EC_SW, tako:ecs_pad_1U_no_ring, F.Cu at (162.6, 73.9)
- added SW7: EC_SW, tako:ecs_pad_1U_no_ring, F.Cu at (181.7, 61.9)
- added SW8: EC_SW, tako:ecs_pad_1U_no_ring, F.Cu at (200.7, 55.9)
- added SW9: EC_SW, tako:ecs_pad_1U_no_ring, F.Cu at (219.8, 62.4)
- added U1: STeMCell, tako:ArduinoProMicro, B.Cu at (257.8, 74.3)
- added U2: 74HC4051, Package_SO:SOIC-16_3.9x9.9mm_P1.27mm, F.Cu at (192.1, 101.9)
- added U3: OPA350, Package_SO:SOIC-8_3.9x4.9mm_P1.27mm, F.Cu at (208.6, 101.9)
Routing:
- net COL0_R: track 197.8 -> 0.00 mm, vias 4 -> 0
- net COL0: track 0.00 -> 193.9 mm, vias 0 -> 4
- net COL1_R: track 186.9 -> 0.00 mm, vias 6 -> 0
- net COL1: track 0.00 -> 185.7 mm, vias 0 -> 6
- net COL2_R: track 163.7 -> 0.00 mm, vias 6 -> 0
- net COL2: track 0.00 -> 160.6 mm, vias 0 -> 6
- net COL4: track 0.00 -> 137.4 mm, vias 0 -> 3
- net COL4_R: track 134.5 -> 0.00 mm, vias 3 -> 0
- net Net-(R1-Pad1): track 0.00 -> 123.9 mm, vias 0 -> 5
- net Net-(R101-Pad1): track 123.8 -> 0.00 mm, vias 5 -> 0
- net Net-(R103-Pad2): track 119.3 -> 0.00 mm, vias 5 -> 0
- net Net-(R3-Pad2): track 0.00 -> 119.2 mm, vias 0 -> 5
- net COL3_R: track 108.3 -> 0.00 mm, vias 3 -> 0
- net Net-(R102-Pad2): track 107.5 -> 0.00 mm, vias 5 -> 0
- net Net-(R2-Pad2): track 0.00 -> 107.5 mm, vias 0 -> 5
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- added copper zone on B.Cu, net GND
- added copper zone on F.Cu, net GND
- removed copper zone on B.Cu, net GND_R
- removed copper zone on F.Cu, net GND_R
Other:
- outline, holes or cut-outs redrawn
