File: rev1/pcb/tako_right.kicad_pcb (KiCad board)
At the start: 2 copper layers, 124.7 x 110.4 mm, 61 parts, among them J1 MJ-4PP-9, SW1 EC_SW, SW10 EC_SW, SW11 EC_SW, SW12 EC_SW, SW13 EC_SW, SW14 EC_SW, SW15 EC_SW, SW16 EC_SW, SW17 EC_SW, SW18 EC_SW, SW2 EC_SW, SW3 EC_SW, SW4 EC_SW, SW5 EC_SW, SW6 EC_SW, SW7 EC_SW, SW8 EC_SW, SW9 EC_SW, U1 STeMCell, U2 74HC4051, U3 OPA350

Commit message: updated holes for 4.5mm standoff
Parts:
- removed BAT_HOLE+1: MountingHole_Pad, tako:bat_pin+
- removed BAT_HOLE-1: MountingHole_Pad, tako:bat_pin-
- removed C1, C3: 100n, Capacitor_SMD:C_0805_2012Metric_Pad1.18x1.45mm_HandSolder
- removed C2: 220p, Capacitor_SMD:C_0805_2012Metric_Pad1.18x1.45mm_HandSolder
- removed DISP1: nice!view, tako:nice_view
- removed H1, H10, H11, H12, H13, H14, H19, H2, H3, H4, H5, H6, H7, H8, H9: MountingHole, tako:MountingHole_3.4mm
- removed H15, H16, H17: MountingHole, tako:M2_hole_3.5mm
- removed J1: MJ-4PP-9, tako:TRRS-PJ-320A
- removed JP1: Ext_Res, Resistor_SMD:R_0805_2012Metric_Pad1.20x1.40mm_HandSolder
- removed PSW1: SW_SPDT, tako:SW_SPDT_SMD_PCM12
- removed R1, R2, R3, R4: 100, Resistor_SMD:R_0805_2012Metric_Pad1.20x1.40mm_HandSolder
- removed R10, R5, R6, R7, R8, R9: 100k, Resistor_SMD:R_0805_2012Metric_Pad1.20x1.40mm_HandSolder
- removed R11: 1k, Resistor_SMD:R_0805_2012Metric_Pad1.20x1.40mm_HandSolder
- removed R12: 5.1k, Resistor_SMD:R_0805_2012Metric_Pad1.20x1.40mm_HandSolder
- removed RSW1: Reset, Button_Switch_SMD:Panasonic_EVQPUL_EVQPUC
- removed SW1, SW10, SW11, SW12, SW13, SW14, SW15, SW2, SW3, SW4, SW5, SW6, SW7, SW8, SW9: EC_SW, tako:ecs_pad_1U_no_ring
- removed SW16, SW17, SW18: EC_SW, tako:ecs_pad_1U_no_ring_90deg
- removed U1: STeMCell, tako:ArduinoProMicro
- removed U2: 74HC4051, Package_SO:SOIC-16_3.9x9.9mm_P1.27mm
- removed U3: OPA350, Package_SO:SOIC-8_3.9x4.9mm_P1.27mm
- added BAT_HOLE+101: MountingHole_Pad, tako:bat_pin+, F.Cu at (53.4, 57.8)
- added BAT_HOLE-101: MountingHole_Pad, tako:bat_pin-, F.Cu at (38.2, 57.8)
- added C101: 100n, Capacitor_SMD:C_0805_2012Metric_Pad1.18x1.45mm_HandSolder, F.Cu at (103.7, 95.6)
- added C102: 220p, Capacitor_SMD:C_0805_2012Metric_Pad1.18x1.45mm_HandSolder, F.Cu at (102.8, 101.5)
- added C103: 100n, Capacitor_SMD:C_0805_2012Metric_Pad1.18x1.45mm_HandSolder, F.Cu at (89.6, 97.6)
- added DISP101: nice!view, tako:nice_view, F.Cu at (45.8, 75.9)
- added H101: MountingHole, MountingHole:MountingHole_4.5mm, F.Cu at (140.9, 44.7)
- added H102: MountingHole, MountingHole:MountingHole_4.5mm, F.Cu at (140.9, 64.4)
- added H103: MountingHole, MountingHole:MountingHole_4.5mm, F.Cu at (140.9, 83.4)
- added H104: MountingHole, MountingHole:MountingHole_4.5mm, F.Cu at (121.9, 32.7)
- added H105: MountingHole, MountingHole:MountingHole_4.5mm, F.Cu at (126.9, 95.0)
- added H106: MountingHole, MountingHole:MountingHole_4.5mm, F.Cu at (102.8, 46.4)
- added H107: MountingHole, MountingHole:MountingHole_4.5mm, F.Cu at (102.8, 65.4)
- added H108: MountingHole, MountingHole:MountingHole_4.5mm, F.Cu at (102.8, 87.0)
- added H109: MountingHole, MountingHole:MountingHole_4.5mm, F.Cu at (83.8, 33.2)
- added H110: MountingHole, MountingHole:MountingHole_4.5mm, F.Cu at (64.7, 35.7)
- added H111: MountingHole, MountingHole:MountingHole_4.5mm, F.Cu at (64.7, 55.4)
- added H112: MountingHole, MountingHole:MountingHole_4.5mm, F.Cu at (64.7, 74.4)
- added H113: MountingHole, MountingHole:MountingHole_4.5mm, F.Cu at (64.2, 106.2)
- added H114: MountingHole, MountingHole:MountingHole_4.5mm, F.Cu at (28.9, 117.0)
- added H115: MountingHole, tako:M2_hole_3.5mm, F.Cu at (53.2, 54.5)
- added H116: MountingHole, tako:M2_hole_3.5mm, F.Cu at (38.4, 54.5)
- added H117: MountingHole, tako:M2_hole_3.5mm, F.Cu at (53.2, 97.0)
- added H18: MountingHole, MountingHole:MountingHole_4.5mm, F.Cu at (45.8, 116.7)
- added J101: MJ-4PP-9, tako:TRRS-PJ-320A, F.Cu at (36.7, 97.0)
- added JP101: Ext_Res, Resistor_SMD:R_0805_2012Metric_Pad1.20x1.40mm_HandSolder, F.Cu at (95.9, 95.6)
- added PSW101: SW_SPDT, tako:SW_SPDT_SMD_PCM12, B.Cu at (45.8, 58.1)
- added R101: 100, Resistor_SMD:R_0805_2012Metric_Pad1.20x1.40mm_HandSolder, B.Cu at (45.8, 62.2)
- added R102: 100, Resistor_SMD:R_0805_2012Metric_Pad1.20x1.40mm_HandSolder, B.Cu at (45.8, 64.2)
- added R103: 100, Resistor_SMD:R_0805_2012Metric_Pad1.20x1.40mm_HandSolder, B.Cu at (45.8, 66.1)
- added R104: 100, Resistor_SMD:R_0805_2012Metric_Pad1.20x1.40mm_HandSolder, F.Cu at (62.2, 98.2)
- added R105: 100k, Resistor_SMD:R_0805_2012Metric_Pad1.20x1.40mm_HandSolder, F.Cu at (127.4, 104.0)
- added R106: 100k, Resistor_SMD:R_0805_2012Metric_Pad1.20x1.40mm_HandSolder, F.Cu at (124.1, 100.0)
- added R107: 100k, Resistor_SMD:R_0805_2012Metric_Pad1.20x1.40mm_HandSolder, F.Cu at (111.7, 95.6)
- added R108: 100k, Resistor_SMD:R_0805_2012Metric_Pad1.20x1.40mm_HandSolder, F.Cu at (120.4, 95.6)
- added R109: 100k, Resistor_SMD:R_0805_2012Metric_Pad1.20x1.40mm_HandSolder, F.Cu at (116.1, 95.6)
- added R110: 100k, Resistor_SMD:R_0805_2012Metric_Pad1.20x1.40mm_HandSolder, F.Cu at (95.9, 97.6)
- added R111: 1k, Resistor_SMD:R_0805_2012Metric_Pad1.20x1.40mm_HandSolder, F.Cu at (100.3, 96.6)
- added R112: 5.1k, Resistor_SMD:R_0805_2012Metric_Pad1.20x1.40mm_HandSolder, F.Cu at (60.2, 98.2)
- added RSW101: Reset, Button_Switch_SMD:Panasonic_EVQPUL_EVQPUC, F.Cu at (38.4, 105.2)
- added SW101: EC_SW, tako:ecs_pad_1U_no_ring, F.Cu at (140.9, 54.9)
- added SW102: EC_SW, tako:ecs_pad_1U_no_ring, F.Cu at (121.9, 42.9)
- added SW103: EC_SW, tako:ecs_pad_1U_no_ring, F.Cu at (102.8, 36.9)
- added SW104: EC_SW, tako:ecs_pad_1U_no_ring, F.Cu at (83.8, 43.4)
- added SW105: EC_SW, tako:ecs_pad_1U_no_ring, F.Cu at (64.7, 45.9)
- added SW106: EC_SW, tako:ecs_pad_1U_no_ring, F.Cu at (140.9, 73.9)
- added SW107: EC_SW, tako:ecs_pad_1U_no_ring, F.Cu at (121.9, 61.9)
- added SW108: EC_SW, tako:ecs_pad_1U_no_ring, F.Cu at (102.8, 55.9)
- added SW109: EC_SW, tako:ecs_pad_1U_no_ring, F.Cu at (83.8, 62.4)
- added SW110: EC_SW, tako:ecs_pad_1U_no_ring, F.Cu at (64.7, 64.9)
- added SW111: EC_SW, tako:ecs_pad_1U_no_ring, F.Cu at (140.9, 93.0)
- added SW112: EC_SW, tako:ecs_pad_1U_no_ring, F.Cu at (121.9, 81.0)
- added SW113: EC_SW, tako:ecs_pad_1U_no_ring, F.Cu at (102.8, 75.0)
- added SW114: EC_SW, tako:ecs_pad_1U_no_ring, F.Cu at (83.8, 81.5)
- added SW115: EC_SW, tako:ecs_pad_1U_no_ring, F.Cu at (64.7, 84.0)
- added SW116: EC_SW, tako:ecs_pad_1U_no_ring_90deg, F.Cu at (38.3, 124.0)
- added SW117: EC_SW, tako:ecs_pad_1U_no_ring_90deg, F.Cu at (54.9, 111.5)
- added SW118: EC_SW, tako:ecs_pad_1U_no_ring_90deg, F.Cu at (74.6, 103.3)
- added U101: STeMCell, tako:ArduinoProMicro, B.Cu at (45.8, 74.3)
- added U102: 74HC4051, Package_SO:SOIC-16_3.9x9.9mm_P1.27mm, F.Cu at (111.4, 101.9)
- added U103: OPA350, Package_SO:SOIC-8_3.9x4.9mm_P1.27mm, F.Cu at (94.9, 101.9)
Routing:
- net COL0_R: track 0.00 -> 197.8 mm, vias 0 -> 4
- net COL0: track 193.9 -> 0.00 mm, vias 4 -> 0
- net COL1_R: track 0.00 -> 186.2 mm, vias 0 -> 6
- net COL1: track 185.7 -> 0.00 mm, vias 6 -> 0
- net COL2_R: track 0.00 -> 163.7 mm, vias 0 -> 6
- net COL2: track 160.6 -> 0.00 mm, vias 6 -> 0
- net COL4: track 137.4 -> 0.00 mm, vias 3 -> 0
- net COL4_R: track 0.00 -> 134.5 mm, vias 0 -> 3
- net Net-(R1-Pad1): track 123.9 -> 0.00 mm, vias 5 -> 0
- net Net-(R101-Pad1): track 0.00 -> 123.8 mm, vias 0 -> 5
- net Net-(R103-Pad2): track 0.00 -> 119.3 mm, vias 0 -> 5
- net Net-(R3-Pad2): track 119.2 -> 0.00 mm, vias 5 -> 0
- net COL3_R: track 0.00 -> 108.3 mm, vias 0 -> 3
- net Net-(R102-Pad2): track 0.00 -> 107.5 mm, vias 0 -> 5
- net Net-(R2-Pad2): track 107.5 -> 0.00 mm, vias 5 -> 0
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- added copper zone on B.Cu, net GND_R
- added copper zone on F.Cu, net GND_R
- removed copper zone on B.Cu, net GND
- removed copper zone on F.Cu, net GND
Other:
- outline, holes or cut-outs redrawn
